Commit message: Changed frame names in URDF

File: src/edubot_description/urdf/edubot.xacro (robot description, xacro)
@@ -24,5 +24,5 @@
   </collision>
 </link>
-<link name="left_wheel_1">
+<link name="left_wheel">
   <inertial>
     <origin xyz="-3.671446903204126e-06 0.009837728922762912 1.9649811738159384e-06" rpy="0 0 0"/>
@@ -33,5 +33,5 @@
     <origin xyz="0.000521 -0.091514 -0.032993" rpy="0 0 0"/>
     <geometry>
-      <mesh filename="package://edubot_description/meshes/left_wheel_1.stl" scale="0.001 0.001 0.001"/>
+      <mesh filename="package://edubot_description/meshes/left_wheel.stl" scale="0.001 0.001 0.001"/>
     </geometry>
     <material name="silver"/>
@@ -40,9 +40,9 @@
     <origin xyz="0.000521 -0.091514 -0.032993" rpy="0 0 0"/>
     <geometry>
-      <mesh filename="package://edubot_description/meshes/left_wheel_1.stl" scale="0.001 0.001 0.001"/>
+      <mesh filename="package://edubot_description/meshes/left_wheel.stl" scale="0.001 0.001 0.001"/>
     </geometry>
   </collision>
 </link>
-<link name="lidar_1">
+<link name="lidar">
   <inertial>
     <origin xyz="-0.020037183493869598 -0.028105106955607077 0.0238922170664298" rpy="0 0 0"/>
@@ -53,5 +53,5 @@
     <origin xyz="0.037521 -0.085896 -0.169993" rpy="0 0 0"/>
     <geometry>
-      <mesh filename="package://edubot_description/meshes/lidar_1.stl" scale="0.001 0.001 0.001"/>
+      <mesh filename="package://edubot_description/meshes/lidar.stl" scale="0.001 0.001 0.001"/>
     </geometry>
     <material name="silver"/>
@@ -60,9 +60,9 @@
     <origin xyz="0.037521 -0.085896 -0.169993" rpy="0 0 0"/>
     <geometry>
-      <mesh filename="package://edubot_description/meshes/lidar_1.stl" scale="0.001 0.001 0.001"/>
+      <mesh filename="package://edubot_description/meshes/lidar.stl" scale="0.001 0.001 0.001"/>
     </geometry>
   </collision>
 </link>
-<link name="laser_1">
+<link name="base_laser">
   <inertial>
     <origin xyz="2.4505540371921875e-07 2.831249775042677e-07 -0.009000296212421988" rpy="0 0 0"/>
@@ -73,5 +73,5 @@
     <origin xyz="0.057521 -0.043896 -0.223493" rpy="0 0 0"/>
     <geometry>
-      <mesh filename="package://edubot_description/meshes/laser_1.stl" scale="0.001 0.001 0.001"/>
+      <mesh filename="package://edubot_description/meshes/dummy.stl" scale="0.001 0.001 0.001"/>
     </geometry>
     <material name="silver"/>
@@ -80,9 +80,9 @@
     <origin xyz="0.057521 -0.043896 -0.223493" rpy="0 0 0"/>
     <geometry>
-      <mesh filename="package://edubot_description/meshes/laser_1.stl" scale="0.001 0.001 0.001"/>
+      <mesh filename="package://edubot_description/meshes/dummy.stl" scale="0.001 0.001 0.001"/>
     </geometry>
   </collision>
 </link>
-<link name="right_wheel_1">
+<link name="right_wheel">
   <inertial>
     <origin xyz="4.840207803405547e-06 -0.009795033661765276 -2.9621241774691054e-07" rpy="0 0 0"/>
@@ -93,5 +93,5 @@
     <origin xyz="0.000521 0.091486 -0.032993" rpy="0 0 0"/>
     <geometry>
-      <mesh filename="package://edubot_description/meshes/right_wheel_1.stl" scale="0.001 0.001 0.001"/>
+      <mesh filename="package://edubot_description/meshes/right_wheel.stl" scale="0.001 0.001 0.001"/>
     </geometry>
     <material name="silver"/>
@@ -100,5 +100,5 @@
     <origin xyz="0.000521 0.091486 -0.032993" rpy="0 0 0"/>
     <geometry>
-      <mesh filename="package://edubot_description/meshes/right_wheel_1.stl" scale="0.001 0.001 0.001"/>
+      <mesh filename="package://edubot_description/meshes/right_wheel.stl" scale="0.001 0.001 0.001"/>
     </geometry>
   </collision>
@@ -107,5 +107,5 @@
   <origin xyz="-0.000521 0.091514 0.032993" rpy="0 0 0"/>
   <parent link="base_link"/>
-  <child link="left_wheel_1"/>
+  <child link="left_wheel"/>
   <axis xyz="-0.0 1.0 0.0"/>
 </joint>
@@ -113,15 +113,15 @@
   <origin xyz="-0.037521 0.085896 0.169993" rpy="0 0 0"/>
   <parent link="base_link"/>
-  <child link="lidar_1"/>
+  <child link="lidar"/>
 </joint>
 <joint name="lidar2laser" type="fixed">
-  <origin xyz="-0.02 -0.042 0.0535" rpy="0 0 0"/>
-  <parent link="lidar_1"/>
-  <child link="laser_1"/>
+  <origin xyz="-0.02 -0.042 0.0465" rpy="0 0 0"/>
+  <parent link="lidar"/>
+  <child link="base_laser"/>
 </joint>
 <joint name="right_motor" type="continuous">
   <origin xyz="-0.000521 -0.091486 0.032993" rpy="0 0 0"/>
   <parent link="base_link"/>
-  <child link="right_wheel_1"/>
+  <child link="right_wheel"/>
   <axis xyz="0.0 1.0 -0.0"/>
 </joint>

Commit message: Aligned LIDAR frame axis

File: src/edubot_description/urdf/edubot.xacro (robot description, xacro)
@@ -116,5 +116,5 @@
 </joint>
 <joint name="lidar2laser" type="fixed">
-  <origin xyz="-0.02 -0.042 0.0465" rpy="0 0 0"/>
+  <origin xyz="-0.02 -0.042 0.0465" rpy="0 0 1.5707963267948966"/>
   <parent link="lidar"/>
   <child link="base_laser"/>
