Commit message: Made compatible for gazebo

File: src/edubot_description/urdf/edubot.trans.xacro (robot description, xacro)
@@ -11,10 +11,10 @@
   </actuator>
 </transmission>
-<transmission name="Rev62_tran">
+<transmission name="right_motor_tran">
   <type>transmission_interface/SimpleTransmission</type>
-  <joint name="Rev62">
+  <joint name="right_motor">
     <hardwareInterface>hardware_interface/EffortJointInterface</hardwareInterface>
   </joint>
-  <actuator name="Rev62_actr">
+  <actuator name="right_motor_actr">
     <hardwareInterface>hardware_interface/EffortJointInterface</hardwareInterface>
     <mechanicalReduction>1</mechanicalReduction>

File: src/edubot_description/urdf/edubot.xacro (robot description, xacro)
@@ -2,6 +2,6 @@
 <robot name="edubot" xmlns:xacro="http://www.ros.org/wiki/xacro">
 <xacro:include filename="$(find edubot_description)/urdf/materials.xacro" />
-<xacro:include filename="$(find edubot_description)/urdf/edubot.trans" />
-<xacro:include filename="$(find edubot_description)/urdf/edubot.gazebo" />
+<xacro:include filename="$(find edubot_description)/urdf/edubot.trans.xacro" />
+<xacro:include filename="$(find edubot_description)/urdf/edubot.gazebo.xacro" />
 <link name="base_link">
   <inertial>
